File: RPi FS HAT.sch (KiCad schematic (older format))
At the start: 7 parts, among them J1 Raspberry_Pi_2_3, SW1 SW_DPST, U1 DHT22

Commit message: Updated symbol arrangement, done with wiring.
Parts:
- renumbered R3 to R1, R1 to R2, R2 to R3
Connections:
- wire segments 0 -> 32
Changed lines of the file:
@@
 L Switch:SW_DPST SW1
 U 1 1 5B7619BD
-P 6900 4100
-F 0 "SW1" H 6900 4425 50  0000 C CNN
-F 1 "SW_DPST" H 6900 4334 50  0000 C CNN
-F 2 "freetronics_footprints:SW_PUSHBUTTON_PTH" H 6900 4100 50  0001 C CNN
-F 3 "" H 6900 4100 50  0001 C CNN
-	1    6900 4100
+P 3350 3250
+F 0 "SW1" H 3350 3575 50  0000 C CNN
+F 1 "SW_DPST" H 3350 3484 50  0000 C CNN
+F 2 "freetronics_footprints:SW_PUSHBUTTON_PTH" H 3350 3250 50  0001 C CNN
+F 3 "" H 3350 3250 50  0001 C CNN
+	1    3350 3250
 	1    0    0    -1
 $EndComp
 $Comp
+L Device:R R1
+U 1 1 5B761A56
+P 3600 4500
+F 0 "R1" H 3530 4454 50  0000 R CNN
+F 1 "R" H 3530 4545 50  0000 R CNN
+F 2 "Resistor_SMD:R_0805_2012Metric" V 3530 4500 50  0001 C CNN
+F 3 "~" H 3600 4500 50  0001 C CNN
+	1    3600 4500
+	-1   0    0    1
+$EndComp
+$Comp
 L Device:R R3
-U 1 1 5B761A56
-P 7500 4250
-F 0 "R3" H 7570 4296 50  0000 L CNN
-F 1 "R" H 7570 4205 50  0000 L CNN
-F 2 "Resistor_SMD:R_0805_2012Metric" V 7430 4250 50  0001 C CNN
-F 3 "~" H 7500 4250 50  0001 C CNN
-	1    7500 4250
-	1    0    0    -1
+U 1 1 5B761ABB
+P 6850 3650
+F 0 "R3" H 6780 3604 50  0000 R CNN
+F 1 "R" H 6780 3695 50  0000 R CNN
+F 2 "Resistor_SMD:R_0805_2012Metric" V 6780 3650 50  0001 C CNN
+F 3 "~" H 6850 3650 50  0001 C CNN
+	1    6850 3650
+	-1   0    0    1
 $EndComp
 $Comp
 L Device:R R2
-U 1 1 5B761ABB
-P 6850 2950
-F 0 "R2" V 6643 2950 50  0000 C CNN
-F 1 "R" V 6734 2950 50  0000 C CNN
-F 2 "Resistor_SMD:R_0805_2012Metric" V 6780 2950 50  0001 C CNN
-F 3 "~" H 6850 2950 50  0001 C CNN
-	1    6850 2950
+U 1 1 5B761B3B
+P 4300 3200
+F 0 "R2" V 4093 3200 50  0000 C CNN
+F 1 "R" V 4184 3200 50  0000 C CNN
+F 2 "Resistor_SMD:R_0805_2012Metric" V 4230 3200 50  0001 C CNN
+F 3 "~" H 4300 3200 50  0001 C CNN
+	1    4300 3200
 	0    1    1    0
-$EndComp
-$Comp
-L Device:R R1
-U 1 1 5B761B3B
-P 4050 2850
-F 0 "R1" H 4120 2896 50  0000 L CNN
-F 1 "R" H 4120 2805 50  0000 L CNN
-F 2 "Resistor_SMD:R_0805_2012Metric" V 3980 2850 50  0001 C CNN
-F 3 "~" H 4050 2850 50  0001 C CNN
-	1    4050 2850
-	1    0    0    -1
 $EndComp
 $Comp
 L Device:LED D1
 U 1 1 5B761BB7
-P 7250 2950
-F 0 "D1" H 7242 2695 50  0000 C CNN
-F 1 "LED" H 7242 2786 50  0000 C CNN
-F 2 "LED_SMD:LED_0805_2012Metric" H 7250 2950 50  0001 C CNN
-F 3 "~" H 7250 2950 50  0001 C CNN
-	1    7250 2950
-	-1   0    0    1
+P 6850 4100
+F 0 "D1" V 6888 3983 50  0000 R CNN
+F 1 "LED" V 6797 3983 50  0000 R CNN
+F 2 "LED_SMD:LED_0805_2012Metric" H 6850 4100 50  0001 C CNN
+F 3 "~" H 6850 4100 50  0001 C CNN
+	1    6850 4100
+	0    -1   -1   0
 $EndComp
 $Comp
 L Sensor:DHT11 U1
 U 1 1 5B761C54
-P 4150 3500
-F 0 "U1" H 3920 3546 50  0000 R CNN
-F 1 "DHT22" H 3920 3455 50  0000 R CNN
-F 2 "Connector_PinHeader_2.54mm:PinHeader_1x04_P2.54mm_Vertical" H 4300 3750 50  0001 C CNN
-F 3 "http://akizukidenshi.com/download/ds/aosong/DHT11.pdf" H 4300 3750 50  0001 C CNN
-	1    4150 3500
+P 4150 4000
+F 0 "U1" H 3920 4046 50  0000 R CNN
+F 1 "DHT22" H 3920 3955 50  0000 R CNN
+F 2 "Connector_PinHeader_2.54mm:PinHeader_1x04_P2.54mm_Vertical" H 4300 4250 50  0001 C CNN
+F 3 "http://akizukidenshi.com/download/ds/aosong/DHT11.pdf" H 4300 4250 50  0001 C CNN
+	1    4150 4000
 	1    0    0    -1
 $EndComp
+Wire Wire Line
+	6850 3500 6850 3400
+Wire Wire Line
+	6850 3400 6400 3400
+Wire Wire Line
+	6850 3800 6850 3950
+Wire Wire Line
+	6850 4250 6850 5150
+Wire Wire Line
+	6850 5150 5300 5150
+Wire Wire Line
+	5300 5150 5300 5000
+Wire Wire Line
+	4450 4000 4600 4000
+Wire Wire Line
+	4600 4000 4600 3200
+Wire Wire Line
+	4600 3200 4800 3200
+Wire Wire Line
+	4050 3700 4050 3200
+Wire Wire Line
+	4050 2250 5700 2250
+Wire Wire Line
+	5700 2250 5700 2400
+Wire Wire Line
+	4450 3200 4600 3200
+Connection ~ 4600 3200
+Wire Wire Line
+	4150 3200 4050 3200
+Connection ~ 4050 3200
+Wire Wire Line
+	4050 3200 4050 2250
+Wire Wire Line
+	4050 4300 4050 5150
+Wire Wire Line
+	4050 5150 5200 5150
+Wire Wire Line
+	5200 5150 5200 5000
+Wire Wire Line
+	3550 3150 3550 3250
+Wire Wire Line
+	3550 3250 3600 3250
+Wire Wire Line
+	3850 3250 3850 2800
+Wire Wire Line
+	3850 2800 4800 2800
+Connection ~ 3550 3250
+Wire Wire Line
+	3550 3250 3550 3350
+Wire Wire Line
+	3150 3150 3150 3250
+Wire Wire Line
+	3150 3250 3050 3250
+Wire Wire Line
+	3050 3250 3050 2250
+Wire Wire Line
+	3050 2250 4050 2250
+Connection ~ 3150 3250
+Wire Wire Line
+	3150 3250 3150 3350
+Connection ~ 4050 2250
+Wire Wire Line
+	3600 4350 3600 3250
+Connection ~ 3600 3250
+Wire Wire Line
+	3600 3250 3850 3250
+Wire Wire Line
+	3600 4650 3600 5150
+Wire Wire Line
+	3600 5150 4050 5150
+Connection ~ 4050 5150
 $EndSCHEMATC

Commit message: Added PWR_FLG and Unconnected.
Connections:
- wire segments 32 -> 35
- no-connect marks 0 -> 34
Changed lines of the file:
@@
 	6850 4250 6850 5150
 Wire Wire Line
-	6850 5150 5300 5150
+	6850 5150 6550 5150
 Wire Wire Line
 	5300 5150 5300 5000
@@
 Connection ~ 4050 3200
 Wire Wire Line
-	4050 3200 4050 2250
+	4050 3200 4050 2550
 Wire Wire Line
 	4050 4300 4050 5150
 Wire Wire Line
-	4050 5150 5200 5150
+	4050 5150 4450 5150
 Wire Wire Line
 	5200 5150 5200 5000
@@
 	3600 5150 4050 5150
 Connection ~ 4050 5150
+NoConn ~ 6400 2800
+NoConn ~ 6400 2900
+NoConn ~ 6400 3100
+NoConn ~ 6400 3200
+NoConn ~ 6400 3500
+NoConn ~ 6400 3600
+NoConn ~ 6400 3800
+NoConn ~ 6400 3900
+NoConn ~ 6400 4000
+NoConn ~ 6400 4100
+NoConn ~ 6400 4200
+NoConn ~ 6400 4400
+NoConn ~ 6400 4500
+NoConn ~ 5900 5000
+NoConn ~ 5800 5000
+NoConn ~ 5700 5000
+NoConn ~ 5600 5000
+NoConn ~ 5500 5000
+NoConn ~ 5400 5000
+NoConn ~ 4800 4400
+NoConn ~ 4800 4300
+NoConn ~ 4800 4200
+NoConn ~ 4800 4100
+NoConn ~ 4800 4000
+NoConn ~ 4800 3900
+NoConn ~ 4800 3700
+NoConn ~ 4800 3600
+NoConn ~ 4800 3500
+NoConn ~ 4800 3300
+NoConn ~ 4800 3100
+NoConn ~ 4800 2900
+NoConn ~ 5400 2400
+NoConn ~ 5500 2400
+NoConn ~ 5800 2400
+$Comp
+L power:PWR_FLAG #FLG0101
+U 1 1 5B7712B6
+P 4450 5150
+F 0 "#FLG0101" H 4450 5225 50  0001 C CNN
+F 1 "PWR_FLAG" H 4450 5324 50  0000 C CNN
+F 2 "" H 4450 5150 50  0001 C CNN
+F 3 "~" H 4450 5150 50  0001 C CNN
+	1    4450 5150
+	1    0    0    -1
+$EndComp
+Connection ~ 4450 5150
+Wire Wire Line
+	4450 5150 5200 5150
+$Comp
+L power:PWR_FLAG #FLG0102
+U 1 1 5B771306
+P 4050 2550
+F 0 "#FLG0102" H 4050 2625 50  0001 C CNN
+F 1 "PWR_FLAG" V 4050 2678 50  0000 L CNN
+F 2 "" H 4050 2550 50  0001 C CNN
+F 3 "~" H 4050 2550 50  0001 C CNN
+	1    4050 2550
+	0    1    1    0
+$EndComp
+Connection ~ 4050 2550
+Wire Wire Line
+	4050 2550 4050 2250
+$Comp
+L power:PWR_FLAG #FLG0103
+U 1 1 5B77134C
+P 6550 5150
+F 0 "#FLG0103" H 6550 5225 50  0001 C CNN
+F 1 "PWR_FLAG" H 6550 5324 50  0000 C CNN
+F 2 "" H 6550 5150 50  0001 C CNN
+F 3 "~" H 6550 5150 50  0001 C CNN
+	1    6550 5150
+	1    0    0    -1
+$EndComp
+Connection ~ 6550 5150
+Wire Wire Line
+	6550 5150 5300 5150
 $EndSCHEMATC
