File: RPi FS HAT.sch (KiCad schematic (older format))
At the start: 7 parts, among them J1 Raspberry_Pi_2_3, SW1 SW_DPST, U1 DHT22

Commit message: Replaced wires with net labels .
Connections:
- net labels added: 3V3, button_input
- wire segments 29 -> 20
Changed lines of the file:
@@
 U 1 1 5B761933
 P 5600 3700
-F 0 "J1" H 5600 5178 50  0000 C CNN
-F 1 "Raspberry_Pi_2_3" H 5600 5087 50  0000 C CNN
+F 0 "J1" H 6200 5100 50  0000 C CNN
+F 1 "Raspberry_Pi_2_3" H 6250 5000 50  0000 C CNN
 F 2 "Connector_PinHeader_2.54mm:PinHeader_2x08_P2.54mm_Vertical" H 5600 3700 50  0001 C CNN
 F 3 "https://www.raspberrypi.org/documentation/hardware/raspberrypi/schematics/rpi_SCH_3bplus_1p0_reduced.pdf" H 5600 3700 50  0001 C CNN
@@
 L Device:R R1
 U 1 1 5B761A56
-P 3600 4500
-F 0 "R1" H 3530 4454 50  0000 R CNN
-F 1 "R" H 3530 4545 50  0000 R CNN
-F 2 "Resistor_SMD:R_0805_2012Metric" V 3530 4500 50  0001 C CNN
-F 3 "~" H 3600 4500 50  0001 C CNN
-	1    3600 4500
+P 3600 3700
+F 0 "R1" H 3530 3654 50  0000 R CNN
+F 1 "R" H 3530 3745 50  0000 R CNN
+F 2 "Resistor_SMD:R_0805_2012Metric" V 3530 3700 50  0001 C CNN
+F 3 "~" H 3600 3700 50  0001 C CNN
+	1    3600 3700
 	-1   0    0    1
 $EndComp
@@
 	4050 3700 4050 3200
 Wire Wire Line
-	4050 2250 5700 2250
-Wire Wire Line
-	5700 2250 5700 2400
-Wire Wire Line
 	4450 3200 4600 3200
 Connection ~ 4600 3200
 Wire Wire Line
 	4150 3200 4050 3200
-Connection ~ 4050 3200
-Wire Wire Line
-	4050 3200 4050 2550
 Wire Wire Line
 	3550 3150 3550 3250
 Wire Wire Line
 	3550 3250 3600 3250
-Wire Wire Line
-	3850 3250 3850 2800
-Wire Wire Line
-	3850 2800 4800 2800
 Connection ~ 3550 3250
 Wire Wire Line
@@
 Wire Wire Line
 	3150 3250 3050 3250
-Wire Wire Line
-	3050 3250 3050 2250
-Wire Wire Line
-	3050 2250 4050 2250
 Connection ~ 3150 3250
 Wire Wire Line
 	3150 3250 3150 3350
-Connection ~ 4050 2250
-Wire Wire Line
-	3600 4350 3600 3250
-Connection ~ 3600 3250
-Wire Wire Line
-	3600 3250 3850 3250
+Wire Wire Line
+	3600 3550 3600 3250
 NoConn ~ 6400 2800
 NoConn ~ 6400 2900
@@
 L power:PWR_FLAG #FLG0102
 U 1 1 5B771306
-P 4050 2550
-F 0 "#FLG0102" H 4050 2625 50  0001 C CNN
-F 1 "PWR_FLAG" V 4050 2678 50  0000 L CNN
-F 2 "" H 4050 2550 50  0001 C CNN
-F 3 "~" H 4050 2550 50  0001 C CNN
-	1    4050 2550
+P 3400 2350
+F 0 "#FLG0102" H 3400 2425 50  0001 C CNN
+F 1 "PWR_FLAG" V 3400 2478 50  0000 L CNN
+F 2 "" H 3400 2350 50  0001 C CNN
+F 3 "~" H 3400 2350 50  0001 C CNN
+	1    3400 2350
 	0    1    1    0
 $EndComp
-Connection ~ 4050 2550
-Wire Wire Line
-	4050 2550 4050 2250
 $Comp
 L power:GND #PWR0101
@@
 $EndComp
 Wire Wire Line
-	3600 4650 3600 4750
+	3600 3850 3600 4750
 $Comp
 L power:GND #PWR0105
@@
 Wire Wire Line
 	4050 4500 4050 4750
+Text Label 4800 2800 2    50   ~ 0
+button_input
+Text Label 3600 3400 0    50   ~ 0
+button_input
+Text Label 5700 2400 1    50   ~ 0
+3V3
+Text Label 4050 3200 1    50   ~ 0
+3V3
+Text Label 3050 3250 2    50   ~ 0
+3V3
 $EndSCHEMATC

Commit message: Named last few wires.
Connections:
- net labels added: led, sensor_data
Changed lines of the file:
@@
 NoConn ~ 5800 2400
-$Comp
-L power:PWR_FLAG #FLG0102
-U 1 1 5B771306
-P 3400 2350
-F 0 "#FLG0102" H 3400 2425 50  0001 C CNN
-F 1 "PWR_FLAG" V 3400 2478 50  0000 L CNN
-F 2 "" H 3400 2350 50  0001 C CNN
-F 3 "~" H 3400 2350 50  0001 C CNN
-	1    3400 2350
-	0    1    1    0
-$EndComp
 $Comp
 L power:GND #PWR0101
@@
 Text Label 3050 3250 2    50   ~ 0
 3V3
+$Comp
+L power:PWR_FLAG #FLG0102
+U 1 1 5B7662CA
+P 3850 2650
+F 0 "#FLG0102" H 3850 2725 50  0001 C CNN
+F 1 "PWR_FLAG" H 3850 2824 50  0000 C CNN
+F 2 "" H 3850 2650 50  0001 C CNN
+F 3 "~" H 3850 2650 50  0001 C CNN
+	1    3850 2650
+	0    -1   -1   0
+$EndComp
+Text Label 3850 2650 0    50   ~ 0
+3V3
+Text Label 6550 3400 0    50   ~ 0
+led
+Text Label 4600 3800 1    50   ~ 0
+sensor_data
+Text Label 3600 4450 0    50   ~ 0
+GND
 $EndSCHEMATC

Commit message: Extended a wire for clarity.
Connections:
- wire segments 20 -> 21
Changed lines of the file:
@@
 Text Label 5700 2400 1    50   ~ 0
 3V3
-Text Label 4050 3200 1    50   ~ 0
+Text Label 4050 2900 2    50   ~ 0
 3V3
 Text Label 3050 3250 2    50   ~ 0
@@
 Text Label 3600 4450 0    50   ~ 0
 GND
+Connection ~ 4050 3200
+Wire Wire Line
+	4050 2900 4050 3200
 $EndSCHEMATC

Commit message: Extended a wire for clarity #2.
Connections:
- wire segments 21 -> 22
Changed lines of the file:
@@
 L Switch:SW_DPST SW1
 U 1 1 5B7619BD
-P 3350 3250
-F 0 "SW1" H 3350 3575 50  0000 C CNN
-F 1 "SW_DPST" H 3350 3484 50  0000 C CNN
-F 2 "freetronics_footprints:SW_PUSHBUTTON_PTH" H 3350 3250 50  0001 C CNN
-F 3 "" H 3350 3250 50  0001 C CNN
-	1    3350 3250
+P 3100 3250
+F 0 "SW1" H 3100 3575 50  0000 C CNN
+F 1 "SW_DPST" H 3100 3484 50  0000 C CNN
+F 2 "freetronics_footprints:SW_PUSHBUTTON_PTH" H 3100 3250 50  0001 C CNN
+F 3 "" H 3100 3250 50  0001 C CNN
+	1    3100 3250
 	1    0    0    -1
 $EndComp
@@
 L Device:R R1
 U 1 1 5B761A56
-P 3600 3700
-F 0 "R1" H 3530 3654 50  0000 R CNN
-F 1 "R" H 3530 3745 50  0000 R CNN
-F 2 "Resistor_SMD:R_0805_2012Metric" V 3530 3700 50  0001 C CNN
-F 3 "~" H 3600 3700 50  0001 C CNN
-	1    3600 3700
+P 3350 3700
+F 0 "R1" H 3280 3654 50  0000 R CNN
+F 1 "R" H 3280 3745 50  0000 R CNN
+F 2 "Resistor_SMD:R_0805_2012Metric" V 3280 3700 50  0001 C CNN
+F 3 "~" H 3350 3700 50  0001 C CNN
+	1    3350 3700
 	-1   0    0    1
 $EndComp
@@
 	4150 3200 4050 3200
 Wire Wire Line
-	3550 3150 3550 3250
-Wire Wire Line
-	3550 3250 3600 3250
-Connection ~ 3550 3250
-Wire Wire Line
-	3550 3250 3550 3350
-Wire Wire Line
-	3150 3150 3150 3250
-Wire Wire Line
-	3150 3250 3050 3250
-Connection ~ 3150 3250
-Wire Wire Line
-	3150 3250 3150 3350
-Wire Wire Line
-	3600 3550 3600 3250
+	3300 3150 3300 3250
+Wire Wire Line
+	3300 3250 3350 3250
+Connection ~ 3300 3250
+Wire Wire Line
+	3300 3250 3300 3350
+Wire Wire Line
+	2900 3150 2900 3250
+Wire Wire Line
+	2900 3250 2800 3250
+Connection ~ 2900 3250
+Wire Wire Line
+	2900 3250 2900 3350
+Wire Wire Line
+	3350 3550 3350 3250
 NoConn ~ 6400 2800
 NoConn ~ 6400 2900
@@
 L power:GND #PWR0104
 U 1 1 5B764DCA
-P 3600 4750
-F 0 "#PWR0104" H 3600 4500 50  0001 C CNN
-F 1 "GND" H 3605 4577 50  0000 C CNN
-F 2 "" H 3600 4750 50  0001 C CNN
-F 3 "" H 3600 4750 50  0001 C CNN
-	1    3600 4750
-	1    0    0    -1
-$EndComp
-Wire Wire Line
-	3600 3850 3600 4750
+P 3350 4750
+F 0 "#PWR0104" H 3350 4500 50  0001 C CNN
+F 1 "GND" H 3355 4577 50  0000 C CNN
+F 2 "" H 3350 4750 50  0001 C CNN
+F 3 "" H 3350 4750 50  0001 C CNN
+	1    3350 4750
+	1    0    0    -1
+$EndComp
+Wire Wire Line
+	3350 3850 3350 4750
 $Comp
 L power:GND #PWR0105
@@
 Text Label 4800 2800 2    50   ~ 0
 button_input
-Text Label 3600 3400 0    50   ~ 0
+Text Label 3350 3400 0    50   ~ 0
 button_input
 Text Label 5700 2400 1    50   ~ 0
 3V3
-Text Label 4050 2900 2    50   ~ 0
+Text Label 4050 2650 2    50   ~ 0
 3V3
-Text Label 3050 3250 2    50   ~ 0
+Text Label 2800 3250 2    50   ~ 0
 3V3
 $Comp
 L power:PWR_FLAG #FLG0102
 U 1 1 5B7662CA
-P 3850 2650
-F 0 "#FLG0102" H 3850 2725 50  0001 C CNN
-F 1 "PWR_FLAG" H 3850 2824 50  0000 C CNN
-F 2 "" H 3850 2650 50  0001 C CNN
-F 3 "~" H 3850 2650 50  0001 C CNN
-	1    3850 2650
+P 4050 2900
+F 0 "#FLG0102" H 4050 2975 50  0001 C CNN
+F 1 "PWR_FLAG" H 4050 3074 50  0000 C CNN
+F 2 "" H 4050 2900 50  0001 C CNN
+F 3 "~" H 4050 2900 50  0001 C CNN
+	1    4050 2900
 	0    -1   -1   0
 $EndComp
-Text Label 3850 2650 0    50   ~ 0
-3V3
 Text Label 6550 3400 0    50   ~ 0
 led
 Text Label 4600 3800 1    50   ~ 0
 sensor_data
-Text Label 3600 4450 0    50   ~ 0
+Text Label 3350 4450 0    50   ~ 0
 GND
 Connection ~ 4050 3200
 Wire Wire Line
+	4050 2650 4050 2900
+Connection ~ 4050 2900
+Wire Wire Line
 	4050 2900 4050 3200

Commit message: Added comments.
Parts:
- R1, R2: value R -> 10KΩ
- R3: value R -> 330Ω
Other:
- note added: "Indicator LED"
- note added: "Momentary button"
- note added: "Sensor"
Changed lines of the file:
@@
 U 1 1 5B761933
 P 5600 3700
-F 0 "J1" H 6200 5100 50  0000 C CNN
-F 1 "Raspberry_Pi_2_3" H 6250 5000 50  0000 C CNN
+F 0 "J1" H 4950 4950 50  0000 C CNN
+F 1 "Raspberry_Pi_2_3" H 6200 4950 50  0000 C CNN
 F 2 "Connector_PinHeader_2.54mm:PinHeader_2x08_P2.54mm_Vertical" H 5600 3700 50  0001 C CNN
 F 3 "https://www.raspberrypi.org/documentation/hardware/raspberrypi/schematics/rpi_SCH_3bplus_1p0_reduced.pdf" H 5600 3700 50  0001 C CNN
@@
 L Switch:SW_DPST SW1
 U 1 1 5B7619BD
-P 3100 3250
-F 0 "SW1" H 3100 3575 50  0000 C CNN
-F 1 "SW_DPST" H 3100 3484 50  0000 C CNN
-F 2 "freetronics_footprints:SW_PUSHBUTTON_PTH" H 3100 3250 50  0001 C CNN
-F 3 "" H 3100 3250 50  0001 C CNN
-	1    3100 3250
+P 2900 3250
+F 0 "SW1" H 2900 3575 50  0000 C CNN
+F 1 "SW_DPST" H 2900 3484 50  0000 C CNN
+F 2 "freetronics_footprints:SW_PUSHBUTTON_PTH" H 2900 3250 50  0001 C CNN
+F 3 "" H 2900 3250 50  0001 C CNN
+	1    2900 3250
 	1    0    0    -1
 $EndComp
@@
 L Device:R R1
 U 1 1 5B761A56
-P 3350 3700
-F 0 "R1" H 3280 3654 50  0000 R CNN
-F 1 "R" H 3280 3745 50  0000 R CNN
-F 2 "Resistor_SMD:R_0805_2012Metric" V 3280 3700 50  0001 C CNN
-F 3 "~" H 3350 3700 50  0001 C CNN
-	1    3350 3700
+P 3150 3700
+F 0 "R1" H 3080 3654 50  0000 R CNN
+F 1 "10KΩ" H 3080 3745 50  0000 R CNN
+F 2 "Resistor_SMD:R_0805_2012Metric" V 3080 3700 50  0001 C CNN
+F 3 "~" H 3150 3700 50  0001 C CNN
+	1    3150 3700
 	-1   0    0    1
 $EndComp
@@
 P 6850 3650
 F 0 "R3" H 6780 3604 50  0000 R CNN
-F 1 "R" H 6780 3695 50  0000 R CNN
+F 1 "330Ω" H 6780 3695 50  0000 R CNN
 F 2 "Resistor_SMD:R_0805_2012Metric" V 6780 3650 50  0001 C CNN
 F 3 "~" H 6850 3650 50  0001 C CNN
@@
 P 4300 3200
 F 0 "R2" V 4093 3200 50  0000 C CNN
-F 1 "R" V 4184 3200 50  0000 C CNN
+F 1 "10KΩ" V 4184 3200 50  0000 C CNN
 F 2 "Resistor_SMD:R_0805_2012Metric" V 4230 3200 50  0001 C CNN
 F 3 "~" H 4300 3200 50  0001 C CNN
@@
 P 4150 4000
 F 0 "U1" H 3920 4046 50  0000 R CNN
-F 1 "DHT22" H 3920 3955 50  0000 R CNN
+F 1 "DHT22" H 4350 4250 50  0000 R CNN
 F 2 "Connector_PinHeader_2.54mm:PinHeader_1x04_P2.54mm_Vertical" H 4300 4250 50  0001 C CNN
 F 3 "http://akizukidenshi.com/download/ds/aosong/DHT11.pdf" H 4300 4250 50  0001 C CNN
@@
 	4150 3200 4050 3200
 Wire Wire Line
-	3300 3150 3300 3250
-Wire Wire Line
-	3300 3250 3350 3250
-Connection ~ 3300 3250
-Wire Wire Line
-	3300 3250 3300 3350
-Wire Wire Line
-	2900 3150 2900 3250
-Wire Wire Line
-	2900 3250 2800 3250
-Connection ~ 2900 3250
-Wire Wire Line
-	2900 3250 2900 3350
-Wire Wire Line
-	3350 3550 3350 3250
+	3100 3150 3100 3250
+Wire Wire Line
+	3100 3250 3150 3250
+Connection ~ 3100 3250
+Wire Wire Line
+	3100 3250 3100 3350
+Wire Wire Line
+	2700 3150 2700 3250
+Wire Wire Line
+	2700 3250 2600 3250
+Connection ~ 2700 3250
+Wire Wire Line
+	2700 3250 2700 3350
+Wire Wire Line
+	3150 3550 3150 3250
 NoConn ~ 6400 2800
 NoConn ~ 6400 2900
@@
 L power:GND #PWR0104
 U 1 1 5B764DCA
-P 3350 4750
-F 0 "#PWR0104" H 3350 4500 50  0001 C CNN
-F 1 "GND" H 3355 4577 50  0000 C CNN
-F 2 "" H 3350 4750 50  0001 C CNN
-F 3 "" H 3350 4750 50  0001 C CNN
-	1    3350 4750
-	1    0    0    -1
-$EndComp
-Wire Wire Line
-	3350 3850 3350 4750
+P 3150 4750
+F 0 "#PWR0104" H 3150 4500 50  0001 C CNN
+F 1 "GND" H 3155 4577 50  0000 C CNN
+F 2 "" H 3150 4750 50  0001 C CNN
+F 3 "" H 3150 4750 50  0001 C CNN
+	1    3150 4750
+	1    0    0    -1
+$EndComp
+Wire Wire Line
+	3150 3850 3150 4750
 $Comp
 L power:GND #PWR0105
@@
 Text Label 4800 2800 2    50   ~ 0
 button_input
-Text Label 3350 3400 0    50   ~ 0
+Text Label 3150 3400 0    50   ~ 0
 button_input
 Text Label 5700 2400 1    50   ~ 0
@@
 Text Label 4050 2650 2    50   ~ 0
 3V3
-Text Label 2800 3250 2    50   ~ 0
+Text Label 2600 3250 2    50   ~ 0
 3V3
 $Comp
@@
 Text Label 4600 3800 1    50   ~ 0
 sensor_data
-Text Label 3350 4450 0    50   ~ 0
+Text Label 3150 4450 0    50   ~ 0
 GND
 Connection ~ 4050 3200
@@
 Wire Wire Line
 	4050 2900 4050 3200
+Wire Notes Line
+	3650 2800 3650 5000
+Wire Notes Line
+	2400 2800 2400 5000
+Wire Notes Line
+	2400 2800 3650 2800
+Wire Notes Line
+	2400 5000 3650 5000
+Text Notes 2400 2800 0    50   ~ 0
+Momentary button
+Wire Notes Line
+	6500 3250 6500 4700
+Wire Notes Line
+	6500 4700 7200 4700
+Wire Notes Line
+	7200 4700 7200 3250
+Wire Notes Line
+	7200 3250 6500 3250
+Text Notes 6550 3250 0    50   ~ 0
+Indicator LED
+Wire Notes Line
+	3700 5000 4700 5000
+Wire Notes Line
+	4700 5000 4700 2500
+Wire Notes Line
+	4700 2500 3700 2500
+Wire Notes Line
+	3700 2500 3700 5000
+Text Notes 3700 2500 0    50   ~ 0
+Sensor
 $EndSCHEMATC

Commit message: Added new symbols.
Parts:
- added D2: LED, LED_SMD:LED_0805_2012Metric, symbol Device:LED
- added R4: 330Ω, Resistor_SMD:R_0805_2012Metric, symbol Device:R
Connections:
- wire segments 22 -> 25
Other:
- note added: "Power Indicator LED"
Changed lines of the file:
@@
 Text Notes 3700 2500 0    50   ~ 0
 Sensor
+$Comp
+L Device:R R4
+U 1 1 5B84AFC3
+P 7850 3150
+F 0 "R4" H 7780 3104 50  0000 R CNN
+F 1 "330Ω" H 7780 3195 50  0000 R CNN
+F 2 "Resistor_SMD:R_0805_2012Metric" V 7780 3150 50  0001 C CNN
+F 3 "~" H 7850 3150 50  0001 C CNN
+	1    7850 3150
+	-1   0    0    1
+$EndComp
+$Comp
+L Device:LED D2
+U 1 1 5B84AFC9
+P 7850 3600
+F 0 "D2" V 7888 3483 50  0000 R CNN
+F 1 "LED" V 7797 3483 50  0000 R CNN
+F 2 "LED_SMD:LED_0805_2012Metric" H 7850 3600 50  0001 C CNN
+F 3 "~" H 7850 3600 50  0001 C CNN
+	1    7850 3600
+	0    -1   -1   0
+$EndComp
+Wire Wire Line
+	7850 3000 7850 2900
+Wire Wire Line
+	7850 3300 7850 3450
+$Comp
+L power:GND #PWR01
+U 1 1 5B84AFD2
+P 7850 3900
+F 0 "#PWR01" H 7850 3650 50  0001 C CNN
+F 1 "GND" H 7855 3727 50  0000 C CNN
+F 2 "" H 7850 3900 50  0001 C CNN
+F 3 "" H 7850 3900 50  0001 C CNN
+	1    7850 3900
+	1    0    0    -1
+$EndComp
+Wire Wire Line
+	7850 3750 7850 3900
+Text Label 7850 2900 2    50   ~ 0
+3V3
+Text Notes 7500 2750 0    50   ~ 0
+Power Indicator LED
+Wire Notes Line
+	7500 2750 7500 4150
+Wire Notes Line
+	7500 4150 8300 4150
+Wire Notes Line
+	8300 4150 8300 2750
+Wire Notes Line
+	8300 2750 7500 2750
 $EndSCHEMATC

Commit message: Added  non-class letter N for fenced in areas.
Other:
- note added: "N1 - Momentary button"
- note added: "N2 - Sensor"
- note added: "N3 - Indicator LED"
- note added: "N4 - \nPower Indicator LED"
- note removed: "Indicator LED"
- note removed: "Momentary button"
- note removed: "Power Indicator LED"
- note removed: "Sensor"
Changed lines of the file:
@@
 	2400 5000 3650 5000
 Text Notes 2400 2800 0    50   ~ 0
-Momentary button
+N1 - Momentary button
 Wire Notes Line
 	6500 3250 6500 4700
@@
 	7200 3250 6500 3250
 Text Notes 6550 3250 0    50   ~ 0
-Indicator LED
+N3 - Indicator LED
 Wire Notes Line
 	3700 5000 4700 5000
@@
 	3700 2500 3700 5000
 Text Notes 3700 2500 0    50   ~ 0
-Sensor
+N2 - Sensor
 $Comp
 L Device:R R4
@@
 3V3
 Text Notes 7500 2750 0    50   ~ 0
-Power Indicator LED
+N4 - \nPower Indicator LED
 Wire Notes Line
 	7500 2750 7500 4150
