File: RPi FS HAT.kicad_pcb (KiCad board)
At the start: 2 copper layers, 27.9 x 17.8 mm, 8 parts, among them J1 Raspberry_Pi_2_3, SW1 SW_DPST, U1 DHT22

Commit message: Completed update of the board.
Parts:
- added D2: LED, LED_SMD:LED_0805_2012Metric, F.Cu at (143.9, 126.6)
- added R4: 330Ω, Resistor_SMD:R_0805_2012Metric, F.Cu at (143.9, 122.5)
Routing:
- net GND: track 34.9 -> 45.9 mm, vias 2 -> 3
- net Net-(D2-Pad2): track 0.00 -> 4.94 mm
- net /3V3: track 31.9 -> 34.5 mm
Other:
- outline, holes or cut-outs redrawn
Changed lines of the file:
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@@
     (thickness 1.6)
     (drawings 22)
-    (tracks 68)
+    (tracks 79)
     (zones 0)
-    (modules 8)
-    (nets 17)
+    (modules 10)
+    (nets 18)
   )
   (page A4)
@@
   (net 15 "Net-(J1-Pad15)")
   (net 16 "Net-(J1-Pad16)")
+  (net 17 "Net-(D2-Pad2)")
   (net_class Default "This is the default net class."
     (clearance 0.2)
@@
     (add_net /sensor_data)
     (add_net "Net-(D1-Pad2)")
+    (add_net "Net-(D2-Pad2)")
     (add_net "Net-(J1-Pad10)")
     (add_net "Net-(J1-Pad12)")
@@
       (xy 1.296529 -1.531292)) (layer B.SilkS) (width 0.01))
   )
+  (module LED_SMD:LED_0805_2012Metric (layer F.Cu)
+    (at 143.8656 126.6444)
+    (descr "LED SMD 0805 (2012 Metric), square (rectangular) end terminal, IPC_7351 nominal, (Body size source: https://docs.google.com/spreadsheets/d/1BsfQQcO9C6DZCsRaXUlFlo91Tg2WpOkGARC1WS5S8t0/edit?usp=sharing), generated with kicad-footprint-generator")
+    (tags diode)
+    (attr smd)
+    (fp_text reference D2 (at 0 -1.65) (layer F.SilkS)
+      (effects (font (size 1 1) (thickness 0.15)))
+    )
+    (fp_text value LED (at 0 1.65) (layer F.Fab)
+      (effects (font (size 1 1) (thickness 0.15)))
+    )
+    (fp_line (start 1 -0.6) (end -0.7 -0.6) (layer F.Fab) (width 0.1))
+    (fp_line (start -0.7 -0.6) (end -1 -0.3) (layer F.Fab) (width 0.1))
+    (fp_line (start -1 -0.3) (end -1 0.6) (layer F.Fab) (width 0.1))
+    (fp_line (start -1 0.6) (end 1 0.6) (layer F.Fab) (width 0.1))
+    (fp_line (start 1 0.6) (end 1 -0.6) (layer F.Fab) (width 0.1))
+    (fp_line (start 1 -0.96) (end -1.685 -0.96) (layer F.SilkS) (width 0.12))
+    (fp_line (start -1.685 -0.96) (end -1.685 0.96) (layer F.SilkS) (width 0.12))
+    (fp_line (start -1.685 0.96) (end 1 0.96) (layer F.SilkS) (width 0.12))
+    (fp_line (start -1.68 0.95) (end -1.68 -0.95) (layer F.CrtYd) (width 0.05))
+    (fp_line (start -1.68 -0.95) (end 1.68 -0.95) (layer F.CrtYd) (width 0.05))
+    (fp_line (start 1.68 -0.95) (end 1.68 0.95) (layer F.CrtYd) (width 0.05))
+    (fp_line (start 1.68 0.95) (end -1.68 0.95) (layer F.CrtYd) (width 0.05))
+    (fp_text user %R (at 0 0) (layer F.Fab)
+      (effects (font (size 0.5 0.5) (thickness 0.08)))
+    )
+    (pad 1 smd roundrect (at -0.9375 0) (size 0.975 1.4) (layers F.Cu F.Paste F.Mask) (roundrect_rratio 0.25)
+      (net 1 GND))
+    (pad 2 smd roundrect (at 0.9375 0) (size 0.975 1.4) (layers F.Cu F.Paste F.Mask) (roundrect_rratio 0.25)
+      (net 17 "Net-(D2-Pad2)"))
+    (model ${KISYS3DMOD}/LED_SMD.3dshapes/LED_0805_2012Metric.wrl
+      (at (xyz 0 0 0))
+      (scale (xyz 1 1 1))
+      (rotate (xyz 0 0 0))
+    )
+  )
+  (module Resistor_SMD:R_0805_2012Metric (layer F.Cu)
+    (at 143.8656 122.4788)
+    (descr "Resistor SMD 0805 (2012 Metric), square (rectangular) end terminal, IPC_7351 nominal, (Body size source: https://docs.google.com/spreadsheets/d/1BsfQQcO9C6DZCsRaXUlFlo91Tg2WpOkGARC1WS5S8t0/edit?usp=sharing), generated with kicad-footprint-generator")
+    (tags resistor)
+    (attr smd)
+    (fp_text reference R4 (at 0 -1.65) (layer F.SilkS)
+      (effects (font (size 1 1) (thickness 0.15)))
+    )
+    (fp_text value 330Ω (at 0 1.65) (layer F.Fab)
+      (effects (font (size 1 1) (thickness 0.15)))
+    )
+    (fp_line (start -1 0.6) (end -1 -0.6) (layer F.Fab) (width 0.1))
+    (fp_line (start -1 -0.6) (end 1 -0.6) (layer F.Fab) (width 0.1))
+    (fp_line (start 1 -0.6) (end 1 0.6) (layer F.Fab) (width 0.1))
+    (fp_line (start 1 0.6) (end -1 0.6) (layer F.Fab) (width 0.1))
+    (fp_line (start -0.258578 -0.71) (end 0.258578 -0.71) (layer F.SilkS) (width 0.12))
+    (fp_line (start -0.258578 0.71) (end 0.258578 0.71) (layer F.SilkS) (width 0.12))
+    (fp_line (start -1.68 0.95) (end -1.68 -0.95) (layer F.CrtYd) (width 0.05))
+    (fp_line (start -1.68 -0.95) (end 1.68 -0.95) (layer F.CrtYd) (width 0.05))
+    (fp_line (start 1.68 -0.95) (end 1.68 0.95) (layer F.CrtYd) (width 0.05))
+    (fp_line (start 1.68 0.95) (end -1.68 0.95) (layer F.CrtYd) (width 0.05))
+    (fp_text user %R (at 0 0) (layer F.Fab)
+      (effects (font (size 0.5 0.5) (thickness 0.08)))
+    )
+    (pad 1 smd roundrect (at -0.9375 0) (size 0.975 1.4) (layers F.Cu F.Paste F.Mask) (roundrect_rratio 0.25)
+      (net 17 "Net-(D2-Pad2)"))
+    (pad 2 smd roundrect (at 0.9375 0) (size 0.975 1.4) (layers F.Cu F.Paste F.Mask) (roundrect_rratio 0.25)
+      (net 3 /3V3))
+    (model ${KISYS3DMOD}/Resistor_SMD.3dshapes/R_0805_2012Metric.wrl
+      (at (xyz 0 0 0))
+      (scale (xyz 1 1 1))
+      (rotate (xyz 0 0 0))
+    )
+  )
+  (gr_line (start 140.208 130.048) (end 140.208 120.65) (layer Edge.Cuts) (width 0.15))
+  (gr_line (start 142.494 131.064) (end 141.224 131.064) (layer Edge.Cuts) (width 0.15))
+  (gr_arc (start 141.224 130.048) (end 140.208 130.048) (angle -90) (layer Edge.Cuts) (width 0.15))
+  (gr_line (start 140.208 119.888) (end 140.208 120.65) (layer Edge.Cuts) (width 0.15))
+  (gr_line (start 146.812 131.064) (end 142.494 131.064) (layer Edge.Cuts) (width 0.15))
   (dimension 17.653 (width 0.3) (layer B.SilkS)
     (gr_text "17.653 mm" (at 172.153 122.1105 270) (layer B.SilkS)
@@
   (gr_line (start 168.148 114.3) (end 168.148 130.048) (layer Edge.Cuts) (width 0.15))
   (gr_line (start 146.812 131.064) (end 167.132 131.064) (layer Edge.Cuts) (width 0.15))
-  (gr_line (start 145.796 121.92) (end 145.796 130.048) (layer Edge.Cuts) (width 0.15))
-  (gr_line (start 141.224 120.904) (end 144.78 120.904) (layer Edge.Cuts) (width 0.15))
   (gr_line (start 140.208 114.808) (end 140.208 119.888) (layer Edge.Cuts) (width 0.15))
   (gr_line (start 167.132 113.284) (end 141.732 113.284) (layer Edge.Cuts) (width 0.15))
   (gr_arc (start 167.132 114.3) (end 168.148 114.3) (angle -90) (layer Edge.Cuts) (width 0.15))
   (gr_arc (start 167.132 130.048) (end 167.132 131.064) (angle -90) (layer Edge.Cuts) (width 0.15))
-  (gr_arc (start 146.812 130.048) (end 145.796 130.048) (angle -90) (layer Edge.Cuts) (width 0.15))
-  (gr_arc (start 144.78 121.92) (end 145.796 121.92) (angle -90) (layer Edge.Cuts) (width 0.15))
-  (gr_arc (start 141.224 119.888) (end 140.208 119.888) (angle -90) (layer Edge.Cuts) (width 0.15))
   (gr_arc (start 141.732 114.808) (end 141.732 113.284) (angle -90) (layer Edge.Cuts) (width 0.15))
   (gr_circle (center 142.621 116.84) (end 141.224 116.84) (layer Edge.Cuts) (width 0.15))
@@
   (segment (start 158.115 119.761) (end 158.115 118.11) (width 0.3) (layer B.Cu) (net 1))
   (segment (start 157.48 120.396) (end 158.115 119.761) (width 0.3) (layer B.Cu) (net 1))
+  (segment (start 142.9281 126.6444) (end 142.9281 125.6561) (width 0.3) (layer F.Cu) (net 1))
+  (via (at 141.732 124.46) (size 1) (drill 0.6) (layers F.Cu B.Cu) (net 1))
+  (segment (start 142.9281 125.6561) (end 141.732 124.46) (width 0.3) (layer F.Cu) (net 1))
+  (segment (start 145.796 120.396) (end 148.336 120.396) (width 0.3) (layer B.Cu) (net 1))
+  (segment (start 141.732 124.46) (end 145.796 120.396) (width 0.3) (layer B.Cu) (net 1))
   (segment (start 166.5455 122.428) (end 166.5455 124.0305) (width 0.25) (layer F.Cu) (net 2))
   (segment (start 166.5455 124.0305) (end 166.116 124.46) (width 0.25) (layer F.Cu) (net 2))
@@
   (segment (start 155.356166 124.018434) (end 154.1272 125.2474) (width 0.3) (layer F.Cu) (net 3))
   (segment (start 155.356166 122.428) (end 155.356166 124.018434) (width 0.3) (layer F.Cu) (net 3))
+  (segment (start 145.3906 122.4788) (end 145.6954 122.174) (width 0.3) (layer F.Cu) (net 3))
+  (segment (start 144.8031 122.4788) (end 145.3906 122.4788) (width 0.3) (layer F.Cu) (net 3))
+  (segment (start 145.6954 121.5196) (end 146.32101 120.89399) (width 0.3) (layer F.Cu) (net 3))
+  (segment (start 145.6954 122.174) (end 145.6954 121.5196) (width 0.3) (layer F.Cu) (net 3))
   (segment (start 160.930832 121.628) (end 160.206832 120.904) (width 0.25) (layer F.Cu) (net 8))
   (segment (start 160.930832 122.428) (end 160.930832 121.628) (width 0.25) (layer F.Cu) (net 8))
@@
   (segment (start 162.015999 119.470999) (end 161.504999 118.959999) (width 0.25) (layer B.Cu) (net 11))
   (segment (start 164.501001 119.951999) (end 164.020001 119.470999) (width 0.25) (layer B.Cu) (net 11))
+  (segment (start 142.9281 124.7694) (end 144.8031 126.6444) (width 0.25) (layer F.Cu) (net 17))
+  (segment (start 142.9281 122.4788) (end 142.9281 124.7694) (width 0.25) (layer F.Cu) (net 17))
   (zone (net 1) (net_name GND) (layer B.Cu) (hatch edge 0.508)
     (connect_pads (clearance 0.54))
